File: vactrolcrossfader.brd (EAGLE design)
At the start: 27.9 x 80.5 mm, 56 parts, among them U1 TL072_SMD

Commit message: v1.2 first commit
Parts:
- removed VR1, VR4: 20k, MusicThingModular:BOURNS_3362P_TRIMMER
- added VR2, VR3: 25k, MusicThingModular:9MM_SNAP-IN_POT
- D3, D4, D5, D6: value (none) -> 3mm led
- R14, R2: value 1k -> 10k
- T1, T2, T3, T4: value (none) -> mmbt3904
- U1: value TL072_SMD -> TL072D; device MusicThingModular:SO08 -> linear:SO08
- moved R17 6.35 mm to (26.2, 21.6)
- moved D6 4.02 mm to (25.4, 29.2)
- moved D4 3.81 mm to (25.4, 38.1)
- moved D5 2.84 mm to (2.54, 29.2)
- moved D3 2.54 mm to (2.54, 38.1)
- moved JP2 2.03 mm to (13.8, 75.1)
Connections:
- removed net N$47: C5.1, U1.8
- removed net N$48: C6.2, U1.4
- net GND: now also C5.1, VR2.3, VR3.3; no longer C5.2, VR1.3, VR4.3
- net N$13: now also VR3.2; no longer VR4.2
- net N$33: now also VR2.2; no longer VR1.2
- net VCC: now also C5.2, U1.8, VR2.1, VR3.1; no longer VR1.1, VR4.1
- net VEE: now also C6.2, U1.4
Routing:
- net GND: track 237.4 -> 0.00 mm, vias 1 -> 0
- net VCC: track 152.8 -> 0.00 mm, vias 3 -> 0
- net VEE: track 105.0 -> 0.00 mm, vias 6 -> 0
- net N$11: track 88.5 -> 0.00 mm
- net N$32: track 79.1 -> 0.00 mm, vias 2 -> 0
- net N$33: track 76.1 -> 0.00 mm, vias 1 -> 0
- net N$41: track 72.9 -> 0.00 mm, vias 1 -> 0
- net N$16: track 60.7 -> 0.00 mm, vias 2 -> 0
- net N$12: track 56.4 -> 0.00 mm
- net N$13: track 46.6 -> 0.00 mm
- net N$3: track 46.3 -> 0.00 mm, vias 2 -> 0
- net N$27: track 43.1 -> 0.00 mm
- net N$29: track 38.8 -> 0.00 mm
- net N$35: track 35.1 -> 0.00 mm, vias 3 -> 0
- net N$26: track 33.4 -> 0.00 mm
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Other:
- board size 27.9 x 80.5 mm -> 27.9 x 81.8 mm
- board text added: "Vactrol crossfader by Mads Kjeldgaard. V1.2"
- board text removed: "Vactrol crossfader by Mads Kjeldgaard. V1.1"
